File: ETI-438/ETI-438.kicad_pcb (KiCad board)
At the start: 2 copper layers, 107.3 x 79.4 mm, 58 parts, among them Q1 BD140, Q2 BC557, U1 LM3900, U2 LM339, U3 LM339

Commit message: update ETI-438, make PCB smaller
Parts:
- removed the REF** at (83.8, 76.2)
- removed the REF** at (83.8, 110.5)
- removed the REF** at (86.4, 57.8)
- removed the REF** at (83.8, 70.6)
- added REF**: TestPoint_THTPad_D3.0mm_Drill1.5mm, TestPoint:TestPoint_THTPad_D3.0mm_Drill1.5mm, F.Cu at (88.3, 76.2)
- added REF**: TestPoint_THTPad_D3.0mm_Drill1.5mm, TestPoint:TestPoint_THTPad_D3.0mm_Drill1.5mm, F.Cu at (88.3, 110.5)
- added REF**: TestPoint_THTPad_D3.0mm_Drill1.5mm, TestPoint:TestPoint_THTPad_D3.0mm_Drill1.5mm, F.Cu at (88.9, 57.8)
- added REF**: TestPoint_THTPad_D3.0mm_Drill1.5mm, TestPoint:TestPoint_THTPad_D3.0mm_Drill1.5mm, F.Cu at (88.3, 70.6)
- R1, R10, R11, R12, R13, R14, R15, R16, R17, R18, R19, R2, R20, R21, R22, R3, R4, R5, R6, R7, R8, R9: footprint Resistor_THT:R_Axial_DIN0207_L6.3mm_D2.5mm_P15.24mm_Horizontal -> Resistor_THT:R_Axial_DIN0309_L9.0mm_D3.2mm_P12.70mm_Horizontal
- moved R22 5.08 mm to (88.3, 106.7)
- moved R11 4.95 mm to (88.3, 100.3)
- moved Q1 4.45 mm to (102.9, 115.6)
- moved REF** 4.45 mm to (88.3, 126.4)
- moved C4 2.54 mm to (94.0, 91.4)
- moved R3 2.54 mm to (104.1, 61.6)
- moved R6 2.54 mm to (104.1, 72.4)
- moved R9 2.54 mm to (101.0, 86.4)
- moved U1 2.54 mm to (106.7, 79.4)
- moved C1 2.54 mm to (98.5, 70.6)
- moved R1 2.54 mm to (107.3, 106.7)
- moved R17 2.54 mm to (159.4, 97.2)
- moved R21 2.54 mm to (107.3, 111.8)
- moved R5 2.54 mm to (101.1, 81.3)
- moved R18 1.27 mm to (151.8, 111.1)
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Connections:
- U1 pad 13: Net-(U1-Pad13) -> (no net)
Routing:
- net Net-(Q1-Pad1): track 23.6 -> 18.9 mm
- net Net-(LED8-Pad2): track 102.6 -> 98.1 mm
- net Net-(R18-Pad1): track 22.4 -> 19.4 mm
- net Net-(D2-Pad2): track 8.52 -> 5.72 mm
- net Net-(R14-Pad1): track 24.6 -> 22.0 mm
- net Net-(Q1-Pad3): track 31.8 -> 29.3 mm
- net Net-(C1-Pad1): track 18.4 -> 15.9 mm
- net Net-(R5-Pad1): track 24.4 -> 21.9 mm
- net Net-(R17-Pad1): track 12.2 -> 14.8 mm
- net Net-(C4-Pad2): track 32.1 -> 29.7 mm
- net GND: track 375.1 -> 372.7 mm
- net Net-(C1-Pad2): track 7.11 -> 5.21 mm
- net Net-(D3-Pad2): track 44.2 -> 42.3 mm
- net Net-(R19-Pad1): track 23.8 -> 25.1 mm
- net Net-(R1-Pad2): track 29.8 -> 28.7 mm
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Other:
- board size 107.3 x 79.4 mm -> 102.9 x 79.4 mm
